File: super_cmoy/super_cmoy.kicad_sch (KiCad schematic)
At the start: 0 parts

Commit message: work
Parts:
- added C1, C2: 220pF, symbol Device:C
- added C3, C4: 3.3uF, symbol Device:C
- added C5, C6: 47pF, symbol Device:C
- added J1: AudioJack3_SwitchTR, symbol Connector_Audio:AudioJack3_SwitchTR
- added J2: AudioJack3, symbol Connector_Audio:AudioJack3
- added K1: IM03, symbol Relay:IM03
- added R1, R2: 274R, symbol Device:R
- added R3, R4: 49.9k, symbol Device:R
- added R5, R6, R7, R8: 2k, symbol Device:R
- added RV1: R_Potentiometer_Dual_Separate, symbol Device:R_Potentiometer_Dual_Separate
- added U1: OPA1688IDRGR, Package_SON:Texas_DSG0008A_WSON-8-1EP_2x2mm_P0.5mm_EP0.9x1.6mm_ThermalVias, symbol Amplifier_Operational:OPA1656ID
Connections:
- new net: J1.T, R2.1
- new net: C2.1, R2.2, RV1.4
- new net: C3.2, R3.2, U1.3 (+)
- new net: C6.2, K1.6, R8.1, U1.7
- new net: C6.1, R6.2, R8.2, U1.6 (-)
- new net: C4.2, R4.2, U1.5 (+)
- new net: C5.1, R5.2, R7.2, U1.2 (-)
- new net: C5.2, K1.3, R7.1, U1.1
- new net: C4.1, RV1.5
- new net: C1.1, R1.2, RV1.1
- new net: J1.R, R1.1
- new net: J2.T, K1.4
- new net: J2.R, K1.5
- new net: C3.1, RV1.2
- new net GND: C1.2, C2.2, J1.RN, J1.S, J1.TN, R3.1, R4.1, R5.1, R6.1, RV1.3, RV1.6
